File: board/board.kicad_pcb (KiCad board)
At the start: 2 copper layers, 21 x 13 mm, 1 part

Commit message: initial
Parts:
- added C1: 10uF, Capacitor_SMD:C_1206_3216Metric, F.Cu at (144.4, 100.6)
- added C2: 2.2uF, Capacitor_SMD:C_1206_3216Metric, F.Cu at (144.5, 92.5)
- added C3: 100nF, Capacitor_SMD:C_0603_1608Metric, F.Cu at (150.3, 91.8)
- added C4: d.n.p, Capacitor_SMD:C_0603_1608Metric, F.Cu at (147.2, 91.0)
- added C5: 22uF, Capacitor_SMD:C_0603_1608Metric, F.Cu at (146.4, 99.8)
- added C6: 22uF, Capacitor_SMD:C_0603_1608Metric, F.Cu at (148.0, 99.8)
- added J1: Conn_01x03_Male, Connector_PinHeader_2.54mm:PinHeader_1x03_P2.54mm_Vertical, F.Cu at (141.4, 93.5)
- added J2: 003_power, on_edge:on_edge_2x05_host, F.Cu at (161.0, 96.5)
- added L1: 6.8uH, Inductor_SMD:L_Chilisin_BMRB00060612, F.Cu at (152.3, 97.0)
- added R1: 182k, Resistor_SMD:R_0603_1608Metric, F.Cu at (147.2, 92.5)
- added R2: 62k, Resistor_SMD:R_0603_1608Metric, F.Cu at (147.2, 94.1)
- added R3: 0R, Resistor_SMD:R_0603_1608Metric, F.Cu at (143.8, 96.8)
- added R4: 0R, Resistor_SMD:R_0603_1608Metric, F.Cu at (148.1, 102.2)
- added U1: AP63200WU, Package_TO_SOT_SMD:TSOT-23-6, F.Cu at (146.6, 96.5)
- LOGO1: moved to B.Cu
- moved LOGO1 1.34 mm to (151.1, 98.2), turned to 180 degrees
Routing:
- net /step_down/out: track 0.00 -> 23.8 mm, vias 0 -> 3
- net GND: track 0.00 -> 20.4 mm, vias 0 -> 25
- net /step_down/in: track 0.00 -> 14.2 mm
- net Net-(J2-5V): track 0.00 -> 10.5 mm, vias 0 -> 1
- net /step_down/SW: track 0.00 -> 8.41 mm
- net /step_down/EN: track 0.00 -> 5.76 mm, vias 0 -> 1
- net /step_down/FB: track 0.00 -> 5.26 mm
- net Net-(U1-BST): track 0.00 -> 5.08 mm
- added copper zone on B.Cu, net GND
- added copper zone on F.Cu, net GND
Other:
- outline, holes or cut-outs redrawn
- board text added: "osf.000"
- board text added: "osf.b143.v1.0"
